Commit message: Add files via upload

File: turtlebot3_burger.urdf.xacro (robot description, xacro)
@@ -143,5 +143,5 @@
     <parent link="base_link"/>
     <child link="second_scan"/>
-    <origin xyz="-0.032 -0.1 0.172" rpy="0 0 0"/>
+    <origin xyz="-0.032 0 0.06" rpy="0 0 0"/>
   </joint>
   <link name="second_scan">

Commit message: Add files via upload

File: turtlebot3_burger.urdf.xacro (robot description, xacro)
@@ -116,5 +116,5 @@
     <parent link="base_link"/>
     <child link="base_scan"/>
-    <origin xyz="-0.032 0 0.172" rpy="0 0 0"/>
+    <origin xyz="-0.032 0 0.4" rpy="0 0 0"/>
   </joint>
   <link name="base_scan">
@@ -127,5 +127,5 @@
     </visual>
     <collision>
-      <origin xyz="0.015 0 -0.0065" rpy="0 0 0"/>
+      <origin xyz="0 0 0" rpy="0 0 0"/>
       <geometry>
         <cylinder length="0.0315" radius="0.055"/>
@@ -163,5 +163,5 @@
     <parent link="base_link"/>
     <child link="gripper2_link"/>
-    <origin xyz="0.06 -0.045 0.04" rpy="1.57 0 1.42"/>
+    <origin xyz="0.06 -0.045 0.02" rpy="1.57 0 1.42"/>
   </joint>
   <link name="gripper2_link" type="fixed">
@@ -194,5 +194,5 @@
     </visual>
     <collision>
-      <origin xyz="0.015 0 -0.0065" rpy="0 0 0"/>
+      <origin xyz="0 0 0" rpy="0 0 0"/>
       <geometry>
         <cylinder length="0.0315" radius="0.055"/>

Commit message: Add files via upload

File: turtlebot3_burger.urdf.xacro (robot description, xacro)
@@ -143,5 +143,5 @@
     <parent link="base_link"/>
     <child link="gripper1_link"/>
-    <origin xyz="0.06 0.045 0.04" rpy="1.57 0 1.72"/>
+    <origin xyz="0.06 0.045 0.04" rpy="1.57 0 1.92"/>
   </joint>
   <link name="gripper1_link" type="fixed">
@@ -163,5 +163,5 @@
     <parent link="base_link"/>
     <child link="gripper2_link"/>
-    <origin xyz="0.06 -0.045 0.02" rpy="1.57 0 1.42"/>
+    <origin xyz="0.06 -0.045 0.04" rpy="1.57 0 1.32"/>
   </joint>
   <link name="gripper2_link" type="fixed">
