Commit message: Add files via upload

File: turtlebot3_burger.gazebo.xacro (robot description, xacro)
@@ -42,5 +42,12 @@
     <material>Gazebo/FlatBlack</material>
   </gazebo>
-  <gazebo reference="imu_link">
+  <gazebo reference="gripper1_link">
+    <sensor type="imu" name="imu">
+      <always_on>true</always_on>
+      <visualize>$(arg imu_visual)</visualize>
+    </sensor>
+    <material>Gazebo/FlatBlack</material>
+  </gazebo>
+  <gazebo reference="gripper2_link">
     <sensor type="imu" name="imu">
       <always_on>true</always_on>

File: turtlebot3_burger.urdf.xacro (robot description, xacro)
@@ -140,8 +140,48 @@
     </inertial>
   </link>
+  <joint name="gripper1_joint" type="fixed">
+    <parent link="base_link"/>
+    <child link="gripper1_link"/>
+    <origin xyz="0.06 0.045 0.04" rpy="1.57 0 1.72"/>
+  </joint>
+  <link name="gripper1_link" type="fixed">
+    <visual>
+      <geometry>
+        <cylinder length="0.1" radius="0.005"/>
+      </geometry>
+      <material name="blue">
+        <color rgba="0 0 .8 1"/>
+      </material>
+    </visual>
+    <collision>
+      <geometry>
+        <cylinder length="0.1" radius="0.005"/>
+      </geometry>
+    </collision>
+  </link>
+  <joint name="gripper2_joint" type="fixed">
+    <parent link="base_link"/>
+    <child link="gripper2_link"/>
+    <origin xyz="0.06 -0.045 0.04" rpy="1.57 0 1.42"/>
+  </joint>
+  <link name="gripper2_link" type="fixed">
+    <visual>
+      <geometry>
+        <cylinder length="0.1" radius="0.005"/>
+      </geometry>
+      <material name="blue">
+        <color rgba="0 0 .8 1"/>
+      </material>
+    </visual>
+    <collision>
+      <geometry>
+        <cylinder length="0.1" radius="0.005"/>
+      </geometry>
+    </collision>
+  </link>
   <joint name="scan2_joint" type="fixed">
     <parent link="base_link"/>
     <child link="second_scan"/>
-    <origin xyz="-0.032 0 0.06" rpy="0 0 0"/>
+    <origin xyz="-0.032 0 0.06	" rpy="0 0 0"/>
   </joint>
   <link name="second_scan">

Commit message: Add files via upload

File: turtlebot3_burger.gazebo.xacro (robot description, xacro)
@@ -140,5 +140,5 @@
   <gazebo reference="second_scan">
 	<material>Gazebo/FlatBlack</material>
-    <sensor type="ray" name="lds_lfcd_sensor">
+    <sensor type="ray" name="lds_lfcd_sensor2">
       <pose>0 0 0 0 0 0</pose>
       <visualize>$(arg laser_visual)</visualize>

File: turtlebot3_burger.urdf.xacro (robot description, xacro)
@@ -116,5 +116,5 @@
     <parent link="base_link"/>
     <child link="base_scan"/>
-    <origin xyz="-0.032 0 0.4" rpy="0 0 0"/>
+    <origin xyz="-0.032 0 0.172" rpy="0 0 0"/>
   </joint>
   <link name="base_scan">

Commit message: Add files via upload

File: turtlebot3_burger.gazebo.xacro (robot description, xacro)
@@ -7,6 +7,6 @@
   </gazebo>
   <gazebo reference="wheel_left_link">
-    <mu1>1.0</mu1>
-    <mu2>1.0</mu2>
+    <mu1>0.1</mu1>
+    <mu2>0.1</mu2>
     <kp>500000.0</kp>
     <kd>10.0</kd>

File: turtlebot3_burger.urdf.xacro (robot description, xacro)
@@ -62,5 +62,5 @@
     <parent link="base_link"/>
     <child link="wheel_right_link"/>
-    <origin xyz="0.0 -0.080 0.023" rpy="-1.57 0 0"/>
+    <origin xyz="0.0 -0.08 0.023" rpy="-1.57 0 0"/>
     <axis xyz="0 0 1"/>
   </joint>
