Commit message: Add files via upload

File: robot_files/turtlebot3_burger.urdf.xacro (robot description, xacro)
@@ -18,7 +18,7 @@
     </visual>
     <collision>
-      <origin xyz="-0.032 0 0.070" rpy="0 0 0"/>
-      <geometry>
-        <box size="0.140 0.140 0.143"/>
+      <origin xyz="-0.032 0 0.090" rpy="0 0 0"/>
+      <geometry>
+        <box size="0.140 0.140 0.200"/>
       </geometry>
     </collision>

Commit message: Add files via upload

File: robot_files/turtlebot3_burger.urdf.xacro (robot description, xacro)
@@ -18,7 +18,7 @@
     </visual>
     <collision>
-      <origin xyz="-0.032 0 0.090" rpy="0 0 0"/>
-      <geometry>
-        <box size="0.140 0.140 0.200"/>
+      <origin xyz="-0.032 0 0.120" rpy="0 0 0"/>
+      <geometry>
+        <box size="0.140 0.140 0.240"/>
       </geometry>
     </collision>
